Commit message: Update forkbot.xacro

File: forkbot/urdf/forkbot.xacro (robot description, xacro)
@@ -1,11 +1,5 @@
 <?xml version='1.0'?>
 <robot name="robot" xmlns:xacro="http://www.ros.org/wiki/xacro">
-  <link name="body" />
-  <visual>
-  <origin> rpy="0 0 0" xyz ="0 0 0" />
-    <geometry>
-      <box size="0.3 0.6 0.15" />
-    </geometry>
-  </visual>
+  <link name="body">
   <inertial>
       <mass value="4.4047990875" />
@@ -15,4 +9,10 @@
         izz="0.001434739" />
     </inertial>
+    <visual>
+     <origin xyz="0 0 0" rpy=" 0 0 0"/>
+      <geometry>
+       <box size=".4 .2 .1"/>
+      </geometry>
+   </visual>
   </link>
   <joint name="joint1" type="continuous">
@@ -21,11 +21,11 @@
     <origin xyz="0.15 0.2 0.15" rpy="0 0 0" />
     <geometry>
-      <cylinder> size="0.2 0.5 0.1"
+      <cylinder size="0.2 0.5 0.1"/>
     </geometry>
     <axis xyz="0 0 0" />
   </joint>
-  <link name="armL1" type="fixed"/>
+  <link name="armL1" type="fixed">
   <visual>
-  <origin> rpy="0 0 0" xyz ="0 0 0" />
+  <origin rpy="0 0 0" xyz ="0 0 0" />
     <geometry>
       <cylinder length="0.3" radius="0.025" />
@@ -45,11 +45,11 @@
     <origin xyz="0 0 0" rpy="0 0 0" />
     <geometry>
-      <cylinder> size="0.2 0.5 0.1"
+      <cylinder size="0.2 0.5 0.1"/>
     </geometry>
     <axis xyz="0 0 0" />
   </joint>
-  <link name="armL2" />
+  <link name="armL2">
   <visual>
-  <origin> rpy="0 0 0" xyz ="0 0 0" />
+  <origin rpy="0 0 0" xyz ="0 0 0" />
     <geometry>
       <cylinder length="0.3" radius="0.025" />
@@ -69,11 +69,11 @@
     <origin xyz="0 0 0.3" rpy="0 0 0" />
     <geometry>
-      <cylinder> size="0.2 0.5 0.1"
+      <cylinder size="0.2 0.5 0.1"/>
     </geometry>
     <axis xyz="0 0 0" />
   </joint>
-  <link name="armL3" />
+  <link name="armL3">
   <visual>
-  <origin> rpy="0 0 0" xyz ="0 0 0" />
+  <origin rpy="0 0 0" xyz ="0 0 0" />
     <geometry>
       <cylinder length="0.3" radius="0.025" />
@@ -94,7 +94,7 @@
     <axis xyz="0 0 0" />
   </joint>
-  <link name="fork" />
+  <link name="fork">
   <visual>
-  <origin> rpy="0 0 0" xyz ="0 0 0" />
+  <origin rpy="0 0 0" xyz ="0 0 0" />
     <geometry>
       <box size="0.1 0.1 0.1" />

Commit message: Fixed gazebo robot spawn problem
The problem was that first in the launch file, the robot spawner was called wrong. That is fixed but the robot didn't appeared in Gazebo. This lead to the second problem which is that the inertial part in the URDF file was missing. (URDF consist of two main parts: visual and inertial. With only visual part, you can visualize only in Rviz. To spawn the robot in Gazebo, you need the inertial part also). I took it from the mybot_description. You can make your robot model changes on forkbot.xacro now.

File: forkbot/urdf/forkbot.xacro (robot description, xacro)
@@ -1,111 +1,135 @@
-<?xml version='1.0'?>
-<robot name="robot" xmlns:xacro="http://www.ros.org/wiki/xacro">
-  <link name="body">
-  <inertial>
-      <mass value="4.4047990875" />
-      <origin xyz="-0.000327 0.000908 0.058457"/>
-      <inertia ixx="0.003000703" ixy="0.000000864" ixz="-0.000011312"
-        iyy="0.002974822" iyz="0.000036294"
-        izz="0.001434739" />
+<?xml version="1.0" encoding="UTF-8"?>
+<!--URDF consist of two main parts: visual and inertial. With only visual part, you can visualize only in Rviz. To spawn the robot in Gazebo, you need the inertial part also -->
+<robot name="forkbot_robot" xmlns:xacro="http://www.ros.org/wiki/xacro">
+  <link name='chassis'>
+    <pose>0 0 0.1 0 0 0</pose>
+    <inertial>
+      <mass value="15.0"/>
+      <origin xyz="0.0 0 0.1" rpy=" 0 0 0"/>
+      <inertia
+          ixx="0.1" ixy="0" ixz="0"
+          iyy="0.1" iyz="0"
+          izz="0.1"
+      />
     </inertial>
-    <visual>
-     <origin xyz="0 0 0" rpy=" 0 0 0"/>
+    <collision name='collision'>
       <geometry>
-       <box size=".4 .2 .1"/>
+        <box size=".4 .2 .1"/>
       </geometry>
-   </visual>
+    </collision>
+    <visual name='chassis_visual'>
+      <origin xyz="0 0 0" rpy=" 0 0 0"/>
+      <geometry>
+        <box size=".4 .2 .1"/>
+      </geometry>
+    </visual>
+    <collision name='caster_collision'>
+      <origin xyz="-0.15 0 -0.05" rpy=" 0 0 0"/>
+      <geometry>
+        <sphere radius="0.05"/>
+      </geometry>
+      <surface>
+        <friction>
+          <ode>
+            <mu>0</mu>
+            <mu2>0</mu2>
+            <slip1>1.0</slip1>
+            <slip2>1.0</slip2>
+          </ode>
+        </friction>
+      </surface>
+    </collision>
+    <visual name='caster_visual'>
+      <origin xyz="-0.15 0 -0.05" rpy=" 0 0 0"/>
+      <geometry>
+        <sphere radius="0.05"/>
+      </geometry>
+    </visual>
+    <collision name='caster_front_collision'>
+      <origin xyz="0.15 0 -0.05" rpy=" 0 0 0"/>
+      <geometry>
+        <sphere radius="0.05"/>
+      </geometry>
+      <surface>
+        <friction>
+          <ode>
+            <mu>0</mu>
+            <mu2>0</mu2>
+            <slip1>1.0</slip1>
+            <slip2>1.0</slip2>
+          </ode>
+        </friction>
+      </surface>
+    </collision>
+    <visual name='caster_front_visual'>
+      <origin xyz="0.15 0 -0.05" rpy=" 0 0 0"/>
+      <geometry>
+        <sphere radius="0.05"/>
+      </geometry>
+    </visual>
   </link>
-  <joint name="joint1" type="continuous">
-    <parent link="body"/>
-    <child link="armL1"/>
-    <origin xyz="0.15 0.2 0.15" rpy="0 0 0" />
-    <geometry>
-      <cylinder size="0.2 0.5 0.1"/>
-    </geometry>
-    <axis xyz="0 0 0" />
-  </joint>
-  <link name="armL1" type="fixed">
-  <visual>
-  <origin rpy="0 0 0" xyz ="0 0 0" />
-    <geometry>
-      <cylinder length="0.3" radius="0.025" />
-    </geometry>
-  </visual>
-  <inertial>
-      <mass value="1.4047990875" />
-      <origin xyz="-0.000327 0.000908 0.058457"/>
-      <inertia ixx="0.003000703" ixy="0.000000864" ixz="-0.000011312"
-        iyy="0.002974822" iyz="0.000036294"
-        izz="0.001434739" />
+  <link name="left_wheel">
+    <!--origin xyz="0.1 0.13 0.1" rpy="0 1.5707 1.5707"/-->
+    <collision name="collision">
+      <origin xyz="0 0 0" rpy="0 1.5707 1.5707"/>
+      <geometry>
+        <cylinder radius="0.1" length="0.05"/>
+      </geometry>
+    </collision>
+    <visual name="left_wheel_visual">
+      <origin xyz="0 0 0" rpy="0 1.5707 1.5707"/>
+      <geometry>
+        <cylinder radius="0.1" length="0.05"/>
+      </geometry>
+    </visual>
+    <inertial>
+      <origin xyz="0 0 0" rpy="0 1.5707 1.5707"/>
+      <mass value="5"/>
+      <inertia
+        ixx=".1" ixy="0.0" ixz="0.0"
+        iyy=".1" iyz="0.0"
+        izz=".1"/>
     </inertial>
   </link>
-  <joint name="joint2" type="revolute">
-    <parent link="armL1"/>
-    <child link="armL2"/>
-    <origin xyz="0 0 0" rpy="0 0 0" />
-    <geometry>
-      <cylinder size="0.2 0.5 0.1"/>
-    </geometry>
-    <axis xyz="0 0 0" />
-  </joint>
-  <link name="armL2">
-  <visual>
-  <origin rpy="0 0 0" xyz ="0 0 0" />
-    <geometry>
-      <cylinder length="0.3" radius="0.025" />
-    </geometry>
-  </visual>
-  <inertial>
-      <mass value="1.4047990875" />
-      <origin xyz="-0.000327 0.000908 0.058457"/>
-      <inertia ixx="0.003000703" ixy="0.000000864" ixz="-0.000011312"
-        iyy="0.002974822" iyz="0.000036294"
-        izz="0.001434739" />
+  <link name="right_wheel">
+    <!--origin xyz="0.1 -0.13 0.1" rpy="0 1.5707 1.5707"/-->
+    <collision name="collision">
+      <origin xyz="0 0 0" rpy="0 1.5707 1.5707"/>
+      <geometry>
+        <cylinder radius="0.1" length="0.05"/>
+      </geometry>
+    </collision>
+    <visual name="right_wheel_visual">
+      <origin xyz="0 0 0" rpy="0 1.5707 1.5707"/>
+      <geometry>
+        <cylinder radius="0.1" length="0.05"/>
+      </geometry>
+    </visual>
+    <inertial>
+      <origin xyz="0 0 0" rpy="0 1.5707 1.5707"/>
+      <mass value="5"/>
+      <inertia
+        ixx=".1" ixy="0.0" ixz="0.0"
+        iyy=".1" iyz="0.0"
+        izz=".1"/>
     </inertial>
   </link>
-  <joint name="joint3" type="revolute">
-    <parent link="armL2"/>
-    <child link="armL3"/>
-    <origin xyz="0 0 0.3" rpy="0 0 0" />
-    <geometry>
-      <cylinder size="0.2 0.5 0.1"/>
-    </geometry>
-    <axis xyz="0 0 0" />
+  <joint type="continuous" name="left_wheel_hinge">
+    <origin xyz="0 0.15 0" rpy="0 0 0"/>
+    <!--origin xyz="0.1 0.13 0" rpy="0 1.5707 1.5707"/-->
+    <child link="left_wheel"/>
+    <parent link="chassis"/>
+    <axis xyz="0 1 0" rpy="0 0 0"/>
+    <limit effort="10000" velocity="1000"/>
+    <joint_properties damping="1.0" friction="1.0"/>
   </joint>
-  <link name="armL3">
-  <visual>
-  <origin rpy="0 0 0" xyz ="0 0 0" />
-    <geometry>
-      <cylinder length="0.3" radius="0.025" />
-    </geometry>
-  </visual>
-  <inertial>
-      <mass value="1.4047990875" />
-      <origin xyz="-0.000327 0.000908 0.058457"/>
-      <inertia ixx="0.003000703" ixy="0.000000864" ixz="-0.000011312"
-        iyy="0.002974822" iyz="0.000036294"
-        izz="0.001434739" />
-    </inertial>
-  </link>
-  <joint name="joint4" type="revolute">
-    <parent link="armL3"/>
-    <child link="fork"/>
-    <origin xyz="0 0 0.3" rpy="0 0 0" />
-    <axis xyz="0 0 0" />
+  <joint type="continuous" name="right_wheel_hinge">
+    <origin xyz="0 -0.15 0" rpy="0 0 0"/>
+    <!--origin xyz="0.1 -0.13 0" rpy="0 1.5707 1.5707"/-->
+    <child link="right_wheel"/>
+    <parent link="chassis"/>
+    <axis xyz="0 1 0" rpy="0 0 0"/>
+    <limit effort="10000" velocity="1000"/>
+    <joint_properties damping="1.0" friction="1.0"/>
   </joint>
-  <link name="fork">
-  <visual>
-  <origin rpy="0 0 0" xyz ="0 0 0" />
-    <geometry>
-      <box size="0.1 0.1 0.1" />
-    </geometry>
-  </visual>
-  <inertial>
-      <mass value="1.4047990875" />
-      <origin xyz="-0.000327 0.000908 0.058457"/>
-      <inertia ixx="0.003000703" ixy="0.000000864" ixz="-0.000011312"
-        iyy="0.002974822" iyz="0.000036294"
-        izz="0.001434739" />
-    </inertial>
-  </link>
 </robot>

Commit message: Add files via upload

File: forkbot/urdf/forkbot.xacro (robot description, xacro)
@@ -1,74 +1,154 @@
-<?xml version="1.0" encoding="UTF-8"?>
-<!--URDF consist of two main parts: visual and inertial. With only visual part, you can visualize only in Rviz. To spawn the robot in Gazebo, you need the inertial part also -->
-<robot name="forkbot_robot" xmlns:xacro="http://www.ros.org/wiki/xacro">
-  <link name='chassis'>
-    <pose>0 0 0.1 0 0 0</pose>
-    <inertial>
-      <mass value="15.0"/>
-      <origin xyz="0.0 0 0.1" rpy=" 0 0 0"/>
-      <inertia
-          ixx="0.1" ixy="0" ixz="0"
-          iyy="0.1" iyz="0"
-          izz="0.1"
-      />
-    </inertial>
-    <collision name='collision'>
-      <geometry>
-        <box size=".4 .2 .1"/>
-      </geometry>
-    </collision>
-    <visual name='chassis_visual'>
-      <origin xyz="0 0 0" rpy=" 0 0 0"/>
-      <geometry>
-        <box size=".4 .2 .1"/>
-      </geometry>
-    </visual>
-    <collision name='caster_collision'>
-      <origin xyz="-0.15 0 -0.05" rpy=" 0 0 0"/>
-      <geometry>
-        <sphere radius="0.05"/>
-      </geometry>
-      <surface>
-        <friction>
-          <ode>
-            <mu>0</mu>
-            <mu2>0</mu2>
-            <slip1>1.0</slip1>
-            <slip2>1.0</slip2>
-          </ode>
-        </friction>
-      </surface>
-    </collision>
-    <visual name='caster_visual'>
-      <origin xyz="-0.15 0 -0.05" rpy=" 0 0 0"/>
-      <geometry>
-        <sphere radius="0.05"/>
-      </geometry>
-    </visual>
-    <collision name='caster_front_collision'>
-      <origin xyz="0.15 0 -0.05" rpy=" 0 0 0"/>
-      <geometry>
-        <sphere radius="0.05"/>
-      </geometry>
-      <surface>
-        <friction>
-          <ode>
-            <mu>0</mu>
-            <mu2>0</mu2>
-            <slip1>1.0</slip1>
-            <slip2>1.0</slip2>
-          </ode>
-        </friction>
-      </surface>
-    </collision>
-    <visual name='caster_front_visual'>
-      <origin xyz="0.15 0 -0.05" rpy=" 0 0 0"/>
-      <geometry>
-        <sphere radius="0.05"/>
-      </geometry>
-    </visual>
-  </link>
-  <link name="left_wheel">
-    <!--origin xyz="0.1 0.13 0.1" rpy="0 1.5707 1.5707"/-->
+<?xml version='1.0'?>
+<robot name="robot" xmlns:xacro="http://www.ros.org/wiki/xacro">
+  <link name="body">
+  <inertial>
+      <mass value="4" />
+      <origin xyz="0 0 0"/>
+      <inertia ixx="0.001" ixy="0.0" ixz="0.0"
+        iyy="0.001" iyz="0.0"
+        izz="0.001" />
+    </inertial>
+    <visual>
+     <origin xyz="0 0 0" rpy=" 0 0 0"/>
+      <geometry>
+       <box size="0.3 0.5 0.1"/>
+      </geometry>
+   </visual>
+   <collision name="collision">
+       <geometry>
+          <box size="0.3 0.5 0.1"/>
+       </geometry>
+     </collision>
+  </link>
+  <joint name="joint1" type="revolute">
+    <parent link="body"/>
+    <child link="armL1"/>
+    <origin xyz="0 -0.2 0.1" rpy="0 0 0" />
+    <geometry>
+       <sphere radius="0.05"/>
+     </geometry>
+    <axis xyz="0 0 0" rpy="0 0 0"/>
+    <limit effort="1000.0" lower="-3.14" upper="3.14" velocity="1"/>
+    <joint_properties damping="1.0"/>
+  </joint>
+  <link name="armL1">
+  <visual>
+  <origin rpy="0 0 0" xyz ="0 0 0" />
+    <geometry>
+      <cylinder length="0.3" radius="0.025" />
+    </geometry>
+  </visual>
+  <collision name="collision">
+      <geometry>
+         <cylinder length="0.3" radius="0.025" />
+      </geometry>
+    </collision>
+  <inertial>
+      <mass value="1" />
+      <origin xyz="0 0 0"/>
+      <inertia ixx="0.001" ixy="0.0" ixz="0.0"
+        iyy="0.001" iyz="0.0"
+        izz="0.001" />
+    </inertial>
+  </link>
+  <joint name="joint2" type="revolute">
+    <parent link="armL1"/>
+    <child link="armL2"/>
+    <origin xyz="0 0 0.3" rpy="0 0 0" />
+   <geometry>
+      <sphere radius="0.025"/>
+    </geometry>
+    <axis xyz="0 0 0" />
+    <limit effort="1000.0" lower="-3.14" upper="3.14" velocity="1"/>
+    <joint_properties damping="1.0"/>
+  </joint>
+  <link name="armL2">
+  <visual>
+  <origin rpy="0 0 0" xyz ="0 0 0" />
+    <geometry>
+      <cylinder length="0.3" radius="0.025" />
+    </geometry>
+  </visual>
+  <collision name="collision">
+      <geometry>
+         <cylinder length="0.3" radius="0.025" />
+      </geometry>
+    </collision>
+  <inertial>
+      <mass value="1" />
+      <origin xyz="0 0 0"/>
+      <inertia ixx="0.001" ixy="0.0" ixz="0.0"
+        iyy="0.001" iyz="0.0"
+        izz="0.001" />
+    </inertial>
+  </link>
+  <joint name="joint3" type="revolute">
+    <parent link="armL2"/>
+    <child link="armL3"/>
+    <origin xyz="0 0 0.3" rpy="0 0 0" />
+    <geometry>
+       <sphere radius="0.025"/>
+     </geometry>
+    <axis xyz="0 0 0" />
+    <limit effort="1000.0" lower="-3.14" upper="3.14" velocity="1"/>
+    <joint_properties damping="1.0"/>
+  </joint>
+  <link name="armL3">
+  <visual>
+  <origin rpy="0 0 0" xyz ="0 0 0" />
+    <geometry>
+      <cylinder length="0.3" radius="0.025" />
+    </geometry>
+  </visual>
+  <collision name="collision">
+      <geometry>
+         <cylinder length="0.3" radius="0.025" />
+      </geometry>
+    </collision>
+  <collision>
+      <geometry>
+        <cylinder length="0.3" radius="0.025" />
+      </geometry>
+    </collision>
+  <inertial>
+      <mass value="1" />
+      <origin xyz="0 0 0"/>
+      <inertia ixx="0.001" ixy="0.0" ixz="0.0"
+        iyy="0.001" iyz="0.0"
+        izz="0.001" />
+    </inertial>
+  </link>
+  <joint name="joint4" type="revolute">
+    <parent link="armL3"/>
+    <child link="fork"/>
+    <origin xyz="0 0 0.1" rpy="0 0 0" />
+    <geometry>
+       <sphere radius="0.025"/>
+     </geometry>
+    <axis xyz="0 0 0" />
+    <limit effort="1000.0" lower="-3.14" upper="3.14" velocity="1"/>
+    <joint_properties damping="1.0"/>
+  </joint>
+  <link name="fork">
+  <visual>
+  <origin rpy="0 0 0" xyz ="0 0.1 0" />
+    <geometry>
+      <box size="0.1 0.2 0.01" />
+    </geometry>
+  </visual>
+    <collision name="collision">
+      <geometry>
+           <box size="0.01 0.4 0.01" />
+      </geometry>
+    </collision>
+  <inertial>
+      <mass value="1" />
+      <origin xyz="-0. 0 0"/>
+      <inertia ixx="0.001" ixy="0.0" ixz="0.0"
+        iyy="0.001" iyz="0.0"
+        izz="0.001" />
+    </inertial>
+  </link>
+  <link name="left_backwheel">
     <collision name="collision">
       <origin xyz="0 0 0" rpy="0 1.5707 1.5707"/>
@@ -92,6 +172,27 @@
     </inertial>
   </link>
-  <link name="right_wheel">
-    <!--origin xyz="0.1 -0.13 0.1" rpy="0 1.5707 1.5707"/-->
+  <link name="left_frontwheel">
+    <collision name="collision">
+      <origin xyz="0 0 0" rpy="0 1.5707 1.5707"/>
+      <geometry>
+        <cylinder radius="0.1" length="0.05"/>
+      </geometry>
+    </collision>
+    <visual name="left_wheel_visual">
+      <origin xyz="0 0 0" rpy="0 1.5707 1.5707"/>
+      <geometry>
+        <cylinder radius="0.1" length="0.05"/>
+      </geometry>
+    </visual>
+    <inertial>
+      <origin xyz="0 0 0" rpy="0 1.5707 1.5707"/>
+      <mass value="5"/>
+      <inertia
+        ixx=".1" ixy="0.0" ixz="0.0"
+        iyy=".1" iyz="0.0"
+        izz=".1"/>
+    </inertial>
+  </link>
+  <link name="right_backwheel">
     <collision name="collision">
       <origin xyz="0 0 0" rpy="0 1.5707 1.5707"/>
@@ -115,21 +216,57 @@
     </inertial>
   </link>
-  <joint type="continuous" name="left_wheel_hinge">
-    <origin xyz="0 0.15 0" rpy="0 0 0"/>
-    <!--origin xyz="0.1 0.13 0" rpy="0 1.5707 1.5707"/-->
-    <child link="left_wheel"/>
-    <parent link="chassis"/>
+  <link name="right_frontwheel">
+    <collision name="collision">
+      <origin xyz="0 0 0" rpy="0 1.5707 1.5707"/>
+      <geometry>
+        <cylinder radius="0.1" length="0.05"/>
+      </geometry>
+    </collision>
+    <visual name="right_wheel_visual">
+      <origin xyz="0 0 0" rpy="0 1.5707 1.5707"/>
+      <geometry>
+        <cylinder radius="0.1" length="0.05"/>
+      </geometry>
+    </visual>
+    <inertial>
+      <origin xyz="0 0 0" rpy="0 1.5707 1.5707"/>
+      <mass value="5"/>
+      <inertia
+        ixx=".1" ixy="0.0" ixz="0.0"
+        iyy=".1" iyz="0.0"
+        izz=".1"/>
+    </inertial>
+  </link>
+  <joint type="continuous" name="left_frontwheel_hinge">
+    <origin xyz="-0.15 0.2 0" rpy="0 0 1.5707"/>
+    <child link="left_frontwheel"/>
+    <parent link="body"/>
     <axis xyz="0 1 0" rpy="0 0 0"/>
     <limit effort="10000" velocity="1000"/>
     <joint_properties damping="1.0" friction="1.0"/>
   </joint>
-  <joint type="continuous" name="right_wheel_hinge">
-    <origin xyz="0 -0.15 0" rpy="0 0 0"/>
-    <!--origin xyz="0.1 -0.13 0" rpy="0 1.5707 1.5707"/-->
-    <child link="right_wheel"/>
-    <parent link="chassis"/>
+  <joint type="continuous" name="left_backwheel_hinge">
+    <origin xyz="-0.15 -0.2 0" rpy="0 0 1.5707"/>
+    <child link="left_backwheel"/>
+    <parent link="body"/>
     <axis xyz="0 1 0" rpy="0 0 0"/>
     <limit effort="10000" velocity="1000"/>
     <joint_properties damping="1.0" friction="1.0"/>
   </joint>
+  <joint type="continuous" name="right_frontwheel_hinge">
+    <origin xyz="0.15 0.2 0" rpy="0 0 1.5707"/>
+    <child link="right_frontwheel"/>
+    <parent link="body"/>
+    <axis xyz="1 0 0" rpy="0 0 0"/>
+    <limit effort="10000" velocity="1000"/>
+    <joint_properties damping="1.0" friction="1.0"/>
+  </joint>
+  <joint type="continuous" name="right_backwheel_hinge">
+    <origin xyz="0.15 -0.2 0" rpy="0 0 1.5707"/>
+    <child link="right_backwheel"/>
+    <parent link="body"/>
+    <axis xyz="1 0 0" rpy="0 0 0"/>
+    <limit effort="10000" velocity="1000"/>
+    <joint_properties damping="1.0" friction="1.0"/>
+  </joint>
 </robot>
